Commit message: located ros2_ws

File: install/robot_6dof/share/robot_6dof/urdf/robot_6dof.urdf.xacro (robot description, xacro)
@@ -1 +1,217 @@
-/home/hoang/ros2_ws1/src/robot_6dof/urdf/robot_6dof.urdf.xacro
+<?xml version="1.0"?>
+<robot name="robot_6dof" xmlns:xacro="http://www.ros.org/wiki/xacro">
+  <xacro:property name="mesh_path" value="package://robot_6dof/meshes/" />
+  <xacro:property name="link_color" value="0.79216 0.81961 0.93333 1" />
+  <link name="base_link">
+    <inertial>
+      <origin xyz="6.9648E-05 2.7131E-08 0.01139" rpy="0 0 0" />
+      <mass value="0.54189" />
+      <inertia ixx="0.001226" ixy="-1.0803E-09" ixz="-1.502E-07" iyy="0.0012286" iyz="-2.6389E-10" izz="0.0023945" />
+    </inertial>
+    <visual>
+      <origin xyz="0 0 0" rpy="0 0 0" />
+      <geometry>
+        <mesh filename="${mesh_path}base_link.STL" />
+      </geometry>
+      <material name="white">
+        <color rgba="1 1 1 1" />
+      </material>
+    </visual>
+    <collision>
+      <origin xyz="0 0 0" rpy="0 0 0" />
+      <geometry>
+        <mesh filename="${mesh_path}base_link.STL" />
+      </geometry>
+    </collision>
+  </link>
+  <link name="Link_1">
+    <inertial>
+      <origin xyz="0.032111 -2.3035E-06 -0.041765" rpy="0 0 0" />
+      <mass value="1.2501" />
+      <inertia ixx="0.0027292" ixy="-6.7358E-08" ixz="-0.00080275" iyy="0.0033332" iyz="-5.048E-08" izz="0.0031674" />
+    </inertial>
+    <visual>
+      <origin xyz="0 0 0" rpy="0 0 0" />
+      <geometry>
+        <mesh filename="${mesh_path}Link_1.STL" />
+      </geometry>
+      <material name="blue_grey">
+        <color rgba="${link_color}" />
+      </material>
+    </visual>
+    <collision>
+      <origin xyz="0 0 0" rpy="0 0 0" />
+      <geometry>
+        <mesh filename="${mesh_path}Link_1.STL" />
+      </geometry>
+    </collision>
+  </link>
+  <link name="Link_2">
+    <inertial>
+      <origin xyz="0.0967690452622868 7.9888520782001E-07 -0.000403484304863755" rpy="0 0 0" />
+      <mass value="1.2592115580279" />
+      <inertia ixx="0.00187031756337727" ixy="-2.8648257564185E-08" ixz="0.000435281947158766" iyy="0.00475904821841891" iyz="4.32501012483649E-08" izz="0.0050185794528046" />
+    </inertial>
+    <visual>
+      <origin xyz="0 0 0" rpy="0 0 0" />
+      <geometry>
+        <mesh filename="${mesh_path}Link_2.STL" />
+      </geometry>
+      <material name="blue_grey"/>
+    </visual>
+    <collision>
+      <origin xyz="0 0 0" rpy="0 0 0" />
+      <geometry>
+        <mesh filename="${mesh_path}Link_2.STL" />
+      </geometry>
+    </collision>
+  </link>
+  <link name="Link_3">
+    <inertial>
+      <origin xyz="0.105409999422065 -1.38975531221996E-06 0.00440023413107865" rpy="0 0 0" />
+      <mass value="0.956951585411102" />
+      <inertia ixx="0.000971593548429778" ixy="-4.63179581797583E-05" ixz="-0.000221367435212386" iyy="0.00315823962788167" iyz="-2.59106477302699E-08" izz="0.00325986339284773" />
+    </inertial>
+    <visual>
+      <origin xyz="0 0 0" rpy="0 0 0" />
+      <geometry>
+        <mesh filename="${mesh_path}Link_3.STL" />
+      </geometry>
+      <material name="blue_grey"/>
+    </visual>
+    <collision>
+      <origin xyz="0 0 0" rpy="0 0 0" />
+      <geometry>
+        <mesh filename="${mesh_path}Link_3.STL" />
+      </geometry>
+    </collision>
+  </link>
+  <link name="Link_4">
+    <inertial>
+      <origin xyz="-1.517E-07 -0.021518 0.050883" rpy="0 0 0" />
+      <mass value="0.26222" />
+      <inertia ixx="0.00027461" ixy="-6.3569E-10" ixz="8.2376E-11" iyy="0.00016148" iyz="3.4428E-05" izz="0.00027185" />
+    </inertial>
+    <visual>
+      <origin xyz="0 0 0" rpy="0 0 0" />
+      <geometry>
+        <mesh filename="${mesh_path}Link_4.STL" />
+      </geometry>
+      <material name="blue_grey"/>
+    </visual>
+    <collision>
+      <origin xyz="0 0 0" rpy="0 0 0" />
+      <geometry>
+        <mesh filename="${mesh_path}Link_4.STL" />
+      </geometry>
+    </collision>
+  </link>
+  <link name="Link_5">
+    <inertial>
+      <origin xyz="2.56050163460753E-07 0.0145939451537695 0.0512076511059981" rpy="0 0 0" />
+      <mass value="0.281075718958217" />
+      <inertia ixx="0.000240924546681779" ixy="-6.57951164796267E-10" ixz="-1.71790582313515E-11" iyy="0.000162706484905412" iyz="-2.81907473481584E-05" izz="0.000239187317752223" />
+    </inertial>
+    <visual>
+      <origin xyz="0 0 0" rpy="0 0 0" />
+      <geometry>
+        <mesh filename="${mesh_path}Link_5.STL" />
+      </geometry>
+      <material name="blue_grey"/>
+    </visual>
+    <collision>
+      <origin xyz="0 0 0" rpy="0 0 0" />
+      <geometry>
+        <mesh filename="${mesh_path}Link_5.STL" />
+      </geometry>
+    </collision>
+  </link>
+  <link name="Link_6">
+    <inertial>
+      <origin xyz="-3.18750079002506E-05 -8.526729322611E-11 0.00682113527098754" rpy="0 0 0" />
+      <mass value="0.102485808599363" />
+      <inertia ixx="2.38399727457236E-05" ixy="-1.39025491840001E-13" ixz="-4.22577617421696E-08" iyy="2.38819125270802E-05" iyz="1.25557534769736E-14" izz="3.91604365481194E-05" />
+    </inertial>
+    <visual>
+      <origin xyz="0 0 0" rpy="0 0 0" />
+      <geometry>
+        <mesh filename="${mesh_path}Link_6.STL" />
+      </geometry>
+      <material name="blue_grey"/>
+    </visual>
+    <collision>
+      <origin xyz="0 0 0" rpy="0 0 0" />
+      <geometry>
+        <mesh filename="${mesh_path}Link_6.STL" />
+      </geometry>
+    </collision>
+  </link>
+  <ros2_control name="GazeboSystem" type="system">
+    <hardware>
+      <plugin>gazebo_ros2_control/GazeboSystem</plugin>
+    </hardware>
+    <joint name="Joint_1">
+      <command_interface name="position"/>
+      <state_interface name="position">
+        <param name="initial_value">0.0</param>
+      </state_interface>
+      <state_interface name="velocity"/>
+    </joint>
+    <joint name="Joint_2">
+      <command_interface name="position"/>
+      <state_interface name="position"/>
+      <state_interface name="velocity"/>
+    </joint>
+    <joint name="Joint_3"> <command_interface name="position"/> <state_interface name="position"/> <state_interface name="velocity"/> </joint>
+    <joint name="Joint_4"> <command_interface name="position"/> <state_interface name="position"/> <state_interface name="velocity"/> </joint>
+    <joint name="Joint_5"> <command_interface name="position"/> <state_interface name="position"/> <state_interface name="velocity"/> </joint>
+    <joint name="Joint_6"> <command_interface name="position"/> <state_interface name="position"/> <state_interface name="velocity"/> </joint>
+  </ros2_control>
+  <gazebo>
+    <plugin filename="libgazebo_ros2_control.so" name="gazebo_ros2_control">
+      <parameters>$(find robot_6dof_moveit_config2)/config/ros2_controllers.yaml</parameters>
+    </plugin>
+  </gazebo>
+  <joint name="Joint_1" type="revolute">
+    <origin xyz="0 0 0.1555" rpy="0 0 -0.014125" />
+    <parent link="base_link" />
+    <child link="Link_1" />
+    <axis xyz="0 0 1" />
+    <limit lower="-${pi}" upper="${pi}" effort="10" velocity="10" />
+  </joint>
+  <joint name="Joint_2" type="revolute">
+    <origin xyz="0.1207 0 0" rpy="${pi/2} -0.00020266 ${pi/2}" />
+    <parent link="Link_1" />
+    <child link="Link_2" />
+    <axis xyz="0 0 1" />
+    <limit lower="0" upper="${3*pi/2}" effort="10" velocity="10" />
+  </joint>
+  <joint name="Joint_3" type="revolute">
+    <origin xyz="0.245 0 -0.0945" rpy="0 0 0" />
+    <parent link="Link_2" />
+    <child link="Link_3" />
+    <axis xyz="0 0 1" />
+    <limit lower="0" upper="${3*pi/2}" effort="10" velocity="10" />
+  </joint>
+  <joint name="Joint_4" type="revolute">
+    <origin xyz="0.25 0 0.05" rpy="0 0 -0.0064821" />
+    <parent link="Link_3" />
+    <child link="Link_4" />
+    <axis xyz="0 0 -1" />
+    <limit lower="-${pi}" upper="${pi}" effort="10" velocity="10" />
+  </joint>
+  <joint name="Joint_5" type="revolute">
+    <origin xyz="0 -0.06 0.066" rpy="${pi/2} 0.004011 0" />
+    <parent link="Link_4" />
+    <child link="Link_5" />
+    <axis xyz="0 0 1" />
+    <limit lower="-${pi}" upper="${pi}" effort="10" velocity="10" />
+  </joint>
+  <joint name="Joint_6" type="revolute">
+    <origin xyz="0 0.082001 0.065999" rpy="-1.5842 -1.5637 0.013376" />
+    <parent link="Link_5" />
+    <child link="Link_6" />
+    <axis xyz="0 0 -1" />
+    <limit lower="-${pi}" upper="${pi}" effort="10" velocity="10" />
+  </joint>
+</robot>

File: install/robot_6dof/share/robot_6dof/urdf/robot_6dof.xacro (robot description, xacro)
@@ -1 +1,191 @@
-/home/hoang/ros2_ws1/src/robot_6dof/urdf/robot_6dof.xacro
+<?xml version="1.0"?>
+<robot name="robot_6dof" xmlns:xacro="http://www.ros.org/wiki/xacro">
+  <xacro:property name="mesh_path" value="package://robot_6dof/meshes/" />
+  <xacro:property name="link_color" value="0.79216 0.81961 0.93333 1" />
+  <link name="base_link">
+    <inertial>
+      <origin xyz="6.9648E-05 2.7131E-08 0.01139" rpy="0 0 0" />
+      <mass value="0.54189" />
+      <inertia ixx="0.001226" ixy="-1.0803E-09" ixz="-1.502E-07" iyy="0.0012286" iyz="-2.6389E-10" izz="0.0023945" />
+    </inertial>
+    <visual>
+      <origin xyz="0 0 0" rpy="0 0 0" />
+      <geometry>
+        <mesh filename="${mesh_path}base_link.STL" />
+      </geometry>
+      <material name="white">
+        <color rgba="1 1 1 1" />
+      </material>
+    </visual>
+    <collision>
+      <origin xyz="0 0 0" rpy="0 0 0" />
+      <geometry>
+        <mesh filename="${mesh_path}base_link.STL" />
+      </geometry>
+    </collision>
+  </link>
+  <link name="Link_1">
+    <inertial>
+      <origin xyz="0.032111 -2.3035E-06 -0.041765" rpy="0 0 0" />
+      <mass value="1.2501" />
+      <inertia ixx="0.0027292" ixy="-6.7358E-08" ixz="-0.00080275" iyy="0.0033332" iyz="-5.048E-08" izz="0.0031674" />
+    </inertial>
+    <visual>
+      <origin xyz="0 0 0" rpy="0 0 0" />
+      <geometry>
+        <mesh filename="${mesh_path}Link_1.STL" />
+      </geometry>
+      <material name="blue_grey">
+        <color rgba="${link_color}" />
+      </material>
+    </visual>
+    <collision>
+      <origin xyz="0 0 0" rpy="0 0 0" />
+      <geometry>
+        <mesh filename="${mesh_path}Link_1.STL" />
+      </geometry>
+    </collision>
+  </link>
+  <link name="Link_2">
+    <inertial>
+      <origin xyz="0.0967690452622868 7.9888520782001E-07 -0.000403484304863755" rpy="0 0 0" />
+      <mass value="1.2592115580279" />
+      <inertia ixx="0.00187031756337727" ixy="-2.8648257564185E-08" ixz="0.000435281947158766" iyy="0.00475904821841891" iyz="4.32501012483649E-08" izz="0.0050185794528046" />
+    </inertial>
+    <visual>
+      <origin xyz="0 0 0" rpy="0 0 0" />
+      <geometry>
+        <mesh filename="${mesh_path}Link_2.STL" />
+      </geometry>
+      <material name="blue_grey"/>
+    </visual>
+    <collision>
+      <origin xyz="0 0 0" rpy="0 0 0" />
+      <geometry>
+        <mesh filename="${mesh_path}Link_2.STL" />
+      </geometry>
+    </collision>
+  </link>
+  <link name="Link_3">
+    <inertial>
+      <origin xyz="0.105409999422065 -1.38975531221996E-06 0.00440023413107865" rpy="0 0 0" />
+      <mass value="0.956951585411102" />
+      <inertia ixx="0.000971593548429778" ixy="-4.63179581797583E-05" ixz="-0.000221367435212386" iyy="0.00315823962788167" iyz="-2.59106477302699E-08" izz="0.00325986339284773" />
+    </inertial>
+    <visual>
+      <origin xyz="0 0 0" rpy="0 0 0" />
+      <geometry>
+        <mesh filename="${mesh_path}Link_3.STL" />
+      </geometry>
+      <material name="blue_grey"/>
+    </visual>
+    <collision>
+      <origin xyz="0 0 0" rpy="0 0 0" />
+      <geometry>
+        <mesh filename="${mesh_path}Link_3.STL" />
+      </geometry>
+    </collision>
+  </link>
+  <link name="Link_4">
+    <inertial>
+      <origin xyz="-1.517E-07 -0.021518 0.050883" rpy="0 0 0" />
+      <mass value="0.26222" />
+      <inertia ixx="0.00027461" ixy="-6.3569E-10" ixz="8.2376E-11" iyy="0.00016148" iyz="3.4428E-05" izz="0.00027185" />
+    </inertial>
+    <visual>
+      <origin xyz="0 0 0" rpy="0 0 0" />
+      <geometry>
+        <mesh filename="${mesh_path}Link_4.STL" />
+      </geometry>
+      <material name="blue_grey"/>
+    </visual>
+    <collision>
+      <origin xyz="0 0 0" rpy="0 0 0" />
+      <geometry>
+        <mesh filename="${mesh_path}Link_4.STL" />
+      </geometry>
+    </collision>
+  </link>
+  <link name="Link_5">
+    <inertial>
+      <origin xyz="2.56050163460753E-07 0.0145939451537695 0.0512076511059981" rpy="0 0 0" />
+      <mass value="0.281075718958217" />
+      <inertia ixx="0.000240924546681779" ixy="-6.57951164796267E-10" ixz="-1.71790582313515E-11" iyy="0.000162706484905412" iyz="-2.81907473481584E-05" izz="0.000239187317752223" />
+    </inertial>
+    <visual>
+      <origin xyz="0 0 0" rpy="0 0 0" />
+      <geometry>
+        <mesh filename="${mesh_path}Link_5.STL" />
+      </geometry>
+      <material name="blue_grey"/>
+    </visual>
+    <collision>
+      <origin xyz="0 0 0" rpy="0 0 0" />
+      <geometry>
+        <mesh filename="${mesh_path}Link_5.STL" />
+      </geometry>
+    </collision>
+  </link>
+  <link name="Link_6">
+    <inertial>
+      <origin xyz="-3.18750079002506E-05 -8.526729322611E-11 0.00682113527098754" rpy="0 0 0" />
+      <mass value="0.102485808599363" />
+      <inertia ixx="2.38399727457236E-05" ixy="-1.39025491840001E-13" ixz="-4.22577617421696E-08" iyy="2.38819125270802E-05" iyz="1.25557534769736E-14" izz="3.91604365481194E-05" />
+    </inertial>
+    <visual>
+      <origin xyz="0 0 0" rpy="0 0 0" />
+      <geometry>
+        <mesh filename="${mesh_path}Link_6.STL" />
+      </geometry>
+      <material name="blue_grey"/>
+    </visual>
+    <collision>
+      <origin xyz="0 0 0" rpy="0 0 0" />
+      <geometry>
+        <mesh filename="${mesh_path}Link_6.STL" />
+      </geometry>
+    </collision>
+  </link>
+  <joint name="Joint_1" type="revolute">
+    <origin xyz="0 0 0.1555" rpy="0 0 -0.014125" />
+    <parent link="base_link" />
+    <child link="Link_1" />
+    <axis xyz="0 0 1" />
+    <limit lower="-${pi}" upper="${pi}" effort="10" velocity="10" />
+  </joint>
+  <joint name="Joint_2" type="revolute">
+    <origin xyz="0.1207 0 0" rpy="${pi/2} -0.00020266 ${pi/2}" />
+    <parent link="Link_1" />
+    <child link="Link_2" />
+    <axis xyz="0 0 1" />
+    <limit lower="0" upper="${3*pi/2}" effort="10" velocity="10" />
+  </joint>
+  <joint name="Joint_3" type="revolute">
+    <origin xyz="0.245 0 -0.0945" rpy="0 0 0" />
+    <parent link="Link_2" />
+    <child link="Link_3" />
+    <axis xyz="0 0 1" />
+    <limit lower="0" upper="${3*pi/2}" effort="10" velocity="10" />
+  </joint>
+  <joint name="Joint_4" type="revolute">
+    <origin xyz="0.25 0 0.05" rpy="0 0 -0.0064821" />
+    <parent link="Link_3" />
+    <child link="Link_4" />
+    <axis xyz="0 0 -1" />
+    <limit lower="-${pi}" upper="${pi}" effort="10" velocity="10" />
+  </joint>
+  <joint name="Joint_5" type="revolute">
+    <origin xyz="0 -0.06 0.066" rpy="${pi/2} 0.004011 0" />
+    <parent link="Link_4" />
+    <child link="Link_5" />
+    <axis xyz="0 0 1" />
+    <limit lower="-${pi}" upper="${pi}" effort="10" velocity="10" />
+  </joint>
+  <joint name="Joint_6" type="revolute">
+    <origin xyz="0 0.082001 0.065999" rpy="-1.5842 -1.5637 0.013376" />
+    <parent link="Link_5" />
+    <child link="Link_6" />
+    <axis xyz="0 0 -1" />
+    <limit lower="-${pi}" upper="${pi}" effort="10" velocity="10" />
+  </joint>
+</robot>

File: install/robot_6dof_moveit_config1/share/robot_6dof_moveit_config1/config/robot_6dof.ros2_control.xacro (robot description, xacro)
@@ -1 +1,48 @@
-/home/hoang/ros2_ws1/src/robot_6dof_moveit_config1/config/robot_6dof.ros2_control.xacro
+<?xml version="1.0"?>
+<robot xmlns:xacro="http://www.ros.org/wiki/xacro">
+    <xacro:macro name="robot_6dof_ros2_control" params="name initial_positions_file">
+        <xacro:property name="initial_positions" value="${xacro.load_yaml(initial_positions_file)['initial_positions']}"/>
+        <ros2_control name="${name}" type="system">
+            <hardware>
+                <!-- By default, set up controllers for simulation. This won't work on real hardware -->
+                <plugin>mock_components/GenericSystem</plugin>
+            </hardware>
+            <joint name="Joint_1">
+                <command_interface name="position"/>
+                <state_interface name="position">
+                  <param name="initial_value">${initial_positions['Joint_1']}</param>
+                </state_interface>
+            </joint>
+            <joint name="Joint_2">
+                <command_interface name="position"/>
+                <state_interface name="position">
+                  <param name="initial_value">${initial_positions['Joint_2']}</param>
+                </state_interface>
+            </joint>
+            <joint name="Joint_3">
+                <command_interface name="position"/>
+                <state_interface name="position">
+                  <param name="initial_value">${initial_positions['Joint_3']}</param>
+                </state_interface>
+            </joint>
+            <joint name="Joint_4">
+                <command_interface name="position"/>
+                <state_interface name="position">
+                  <param name="initial_value">${initial_positions['Joint_4']}</param>
+                </state_interface>
+            </joint>
+            <joint name="Joint_5">
+                <command_interface name="position"/>
+                <state_interface name="position">
+                  <param name="initial_value">${initial_positions['Joint_5']}</param>
+                </state_interface>
+            </joint>
+            <joint name="Joint_6">
+                <command_interface name="position"/>
+                <state_interface name="position">
+                  <param name="initial_value">${initial_positions['Joint_6']}</param>
+                </state_interface>
+            </joint>
+        </ros2_control>
+    </xacro:macro>
+</robot>

File: install/robot_6dof_moveit_config1/share/robot_6dof_moveit_config1/config/robot_6dof.urdf.xacro (robot description, xacro)
@@ -1 +1,9 @@
-/home/hoang/ros2_ws1/src/robot_6dof_moveit_config1/config/robot_6dof.urdf.xacro
+<?xml version="1.0"?>
+<robot xmlns:xacro="http://www.ros.org/wiki/xacro" name="robot_6dof">
+    <xacro:arg name="initial_positions_file" default="initial_positions.yaml" />
+    <!-- Import robot_6dof urdf file -->
+    <xacro:include filename="$(find robot_6dof)/urdf/robot_6dof.urdf.xacro" />
+    <!-- Import control_xacro -->
+    <xacro:include filename="robot_6dof.ros2_control.xacro" />
+    <xacro:robot_6dof_ros2_control name="FakeSystem" initial_positions_file="$(arg initial_positions_file)"/>
+</robot>
